File: Hardware/kicad/hack_cube.kicad_sch (KiCad schematic)
At the start: 62 parts, among them IC1 FDC6331L, J1 USB_B_Micro, SW1 SW_DIP_x01, U1 ATmega32U4RC-M, Y1 8MHz

Commit message: update
Parts:
- removed C3: 100n, symbol Device:C
- removed C6: 100n, Capacitor_SMD:C_0805_2012Metric, symbol Device:C
- added C29, C32, C37, C9: 0.1U, symbol Device:C
- added C3: 10U, symbol Device:C_Polarized_Small_US
- added C30, C31, C35: 22U, symbol Device:C
- added C34: 22P, symbol Device:C
- added C36: 2.2U, symbol Device:C
- added C38: 4.7U, symbol Device:C
- added C39, C45, C? (x2): 100n, symbol Device:C
- added C40, C41, C42: C, symbol Device:C
- added C43, C44: 1U, symbol Device:C
- added C? (x2): 22p, symbol Device:C
- added C?: 22u, symbol Device:C_Polarized_Small_US
- added D8: SS34, symbol Device:D
- added D9: LED, symbol Device:LED
- added D?: WS2812, LED_SMD:LED_WS2812_PLCC6_5.0x5.0mm_P1.6mm, symbol LED:WS2812
- added F1, F?: PTCSMD, symbol Device:Polyfuse_Small
- added J?: USB_B_Micro, Connector_USB:USB_Micro-B_Molex-105017-0001, symbol Connector:USB_B_Micro
- added L2, L3: 3.3UH, symbol Device:L
- added L4: 1U, symbol Device:L
- added Q? (x2): S8050, Package_TO_SOT_THT:TO-92_Inline, symbol Transistor_BJT:S8050
- added R10, R11: 22, symbol Device:R
- added R17: 88K, symbol Device:R
- added R18, R?: 12K, symbol Device:R
- added R19: 45K, symbol Device:R
- added R20, R? (x2): 10K, symbol Device:R
- added R21, R24: NC, symbol Device:R
- added R22: 1.25K, symbol Device:R
- added R23: R, symbol Device:R
- added R? (x2): 5.1k, symbol Device:R
- added R?: 12k, symbol Device:R
- added U10: TPS61240, symbol Power_Management:TPS61240
- added U11: LTC4054, symbol Power_Management:LTC4054
- added U12, U13: FP6134-33S5, symbol Power_Management:FP6134-33S5
- added U14: CH340G, Package_SO:SOIC-16_3.9x9.9mm_P1.27mm, symbol Interface_USB:CH340G
- added U8: PW5300, symbol Power_Management:PW5300
- added U9: PW2053, symbol Power_Management:PW2053
- added U?: ESP-12F(ESP8266MOD), kicad_lceda:WIFIM-SMD_ESP-12F-ESP8266MOD, symbol esp8266:ESP-12F(ESP8266MOD)
- added U?: E01-ML01S, kicad_lceda:WIRELM-SMD_E01-ML01S, symbol e01:E01-ML01S
- added U?: E07-M1101S, kicad_lceda:WIRELM-SMD_E07-M1101S, symbol e07:E07-M1101S
- added Y?: Crystal_Small, symbol Device:Crystal_Small
- C4: value 100n -> 0.1U
- C5: value 100n -> 0.1U; footprint Capacitor_SMD:C_0805_2012Metric -> (none)
- C7: value 1U -> 0.1U
- gave numbers to parts that had none: 34
- renumbered Cc8 to C6
Connections:
- net +3V3: now also R1.2, C34.1, C35.1, C44.2, C9.1, D?.3 (VCC), D?.5 (VDD), L3.2, R19.1, R?.1, R?.2, R?.2, R?.2, U13.5 (VOUT), U14.16 (VCC), U14.4 (V3), U?.1 (VCC), U?.1 (VCC), U?.8 (VCC); no longer R1.1
- net +5V: now also C3.1, C31.1, C32.1, C37.2, C38.1, C?.1, D8.1 (K), F1.1, F?.1, R17.1, R21.1, R24.1, U10.2 (VOUT), U10.3 (FB), U11.4 (VCC), U9.1 (CE), U9.4 (VIN); no longer J1.1 (VBUS)
- net Earth: now also SW1.1, C29.2, C3.2, C30.2, C31.2, C32.2, C35.2, C36.2, C37.1, C38.2, C39.2, C40.1, C41.1, C42.2, C43.1, C44.1, C45.2, C9.2, C?.1, C?.1, C?.1, C?.2, C?.2, D?.6 (VSS), J?.5 (GND), R18.2, R20.2, R22.1, U10.1 (GND), U11.2 (GND), U12.2 (GND), U13.2 (GND), U14.1 (GND), U8.2 (GND), U8.6 (OPC), U9.2 (GND), U?.8 (GND), U?.8 (GND), U?.9 (GND); no longer SW1.2
- net RD_N: now also R11.2; no longer J1.3 (D+)
- net RD_P: now also R10.1; no longer J1.2 (D-)
- net AMISO renamed ISP_MOSI
- net ISP_MOSI: now also U?.6 (MISO), U?.6 (MISO/GDO1)
- net AMOSI renamed ISP_MISO
- net ISP_MISO: now also U?.5 (MOSI), U?.5 (MOSI)
- net ASCK renamed ISP_SCK
- net ISP_SCK: now also U?.4 (SCK), U?.4 (SCK)
- removed net RESET: R1.2, SW1.1, U1.13 (~{RESET})
- net XTAL_1: no longer names the net of C1.1, Y1.1
- net XTAL_1: now also U1.16 (XTAL2); no longer U1.17 (XTAL1)
- net XTAL_2: no longer names the net of C2.2, Y1.3
- net XTAL_2: now also U1.17 (XTAL1); no longer U1.16 (XTAL2)
- new net: R22.2, U11.5 (PROG)
- new net: R17.2, R18.1, U8.3 (FB)
- new net: Q?.1 (E), R?.1, U14.14 (~{RTS})
- new net: Q?.2 (B), R?.2 (x2)
- new net: C?.2, R?.1, R?.1, U?.1 (RST), U?.4 (GPIO16)
- new net: C45.1, U13.4 (BP)
- new net: Q?.1 (E), R?.1, U14.13 (~{DTR})
- new net: C?.2, U14.7 (XI), Y?.2
- new net: C?.2, U14.8 (XO), Y?.1
- new net: L3.1, U9.3 (LX)
- new net: C34.2, R19.2, R20.1, U9.5 (FB)
- new net: D8.2 (A), L2.2, U8.1 (LX)
- new net: J1.3 (D+), R11.1
- new net: F1.2, J1.1 (VBUS)
- new net: J1.2 (D-), R10.2
- new net: D9.1 (K), U11.3 (BAT)
- new net: R23.1, U12.3 (SHDN)
- new net: C42.1, U12.4 (BP)
- new net: F?.2, J?.1 (VBUS)
- new net: L4.2, U10.5 (L)
- new net 3.3V_RF: C41.2, U12.5 (VOUT)
- new net 3V~24V: C29.1, C30.1, L2.1, U8.4 (EN), U8.5 (VIN)
- new net A0_NRF_CS: U?.3 (CSN)
- new net A1_NRF_CE: U?.2 (CE)
- new net A2_RF_GDO0: U?.2 (GDO0)
- new net A3_RF_CS: U?.3 (CSN)
- new net ADC: U?.2 (ADC)
- new net ARST: U?.5 (GPIO14)
- new net ARX: U?.10 (GPIO15)
- new net ATX: U?.7 (GPIO13)
- new net BAT: C39.1, U11.1 (CHRG)
- new net BCS: U?.17 (CS0)
- new net BMISO: U?.18 (MISO)
- new net BMOSI: U?.21 (MOSI)
- new net BSCK: U?.22 (SCLK)
- new net CHUD+: J?.3 (D+), U14.5 (UD+)
- new net CHUD-: J?.2 (D-), U14.6 (UD-)
- new net CH_GPIO_0: Q?.3 (C), R?.2, U?.12 (GPIO0)
- new net CH_RST: C?.1, Q?.3 (C), R?.1, U?.3 (EN)
- new net CH_RXD: U14.3 (RXD), U?.16 (TXD0)
- new net CH_TXD: U14.2 (TXD), U?.15 (RXD0)
- new net D2_RF_GDO2: U?.7 (GDO2)
- new net D7_IRQ: U?.7 (IRQ)
- new net EN_LED: U?.6 (GPIO12)
- new net IICSCL: U?.13 (GPIO4)
- new net IICSDA: U?.14 (GPIO5)
- new net ISP_RST: R1.1, SW1.2, U1.13 (~{RESET})
- new net LED: D?.2 (DIN), U?.11 (GPIO2)
- new net POWER_4.2V: C36.1, C40.2, C43.2, L4.1, R21.2, R23.2, R24.2, U10.4 (EN), U10.6 (VIN), U12.1 (VIN), U13.1 (VIN), U13.3 (SHDN)
- no-connect marks 3 -> 14
Other:
- moved on the sheet: C1, C10, C11, C12, C13, C14, C15, C16, C17, C18, C19, C2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

Commit message: [update]
Parts:
- removed C15, C39, C45: 100n, symbol Device:C
- removed C16: 10u, symbol Device:C_Polarized_Small_US
- removed C18, C22, C27: 0.1u, symbol Device:C
- removed C24: 47u, symbol Device:C_Polarized_Small_US
- removed C28: 47n, symbol Device:C
- removed C29, C32, C37: 0.1U, symbol Device:C
- removed C31, C35: 22U, symbol Device:C
- removed C34: 22P, symbol Device:C
- removed C36: 2.2U, symbol Device:C
- removed C38: 4.7U, symbol Device:C
- removed C40, C41, C42: C, symbol Device:C
- removed C43, C44: 1U, symbol Device:C
- removed C8: 100uf, symbol Device:C
- removed C?: 22u, symbol Device:C_Polarized_Small_US
- removed D1, D5, D6, D7, D9: LED, symbol Device:LED
- removed D8: SS34, symbol Device:D
- removed F?: PTCSMD, symbol Device:Polyfuse_Small
- removed IC1: FDC6331L, SSOT6, symbol FDC6331L:FDC6331L
- removed J?: USB_B_Micro, Connector_USB:USB_Micro-B_Molex-105017-0001, symbol Connector:USB_B_Micro
- removed L2, L3: 3.3UH, symbol Device:L
- removed L4: 1U, symbol Device:L
- removed R10, R11: 22, symbol Device:R
- removed R12: 2.2k, symbol Device:R
- removed R13, R6: 10k, symbol Device:R
- removed R14: 130, symbol Device:R
- removed R18: 12K, symbol Device:R
- removed R19: 45K, symbol Device:R
- removed R2, R8: 1k, symbol Device:R
- removed R20: 10K, symbol Device:R
- removed R21, R24: NC, symbol Device:R
- removed R22: 1.25K, symbol Device:R
- removed R23: R, symbol Device:R
- removed R5: 330R, symbol Device:R
- removed SW1: SW_DIP_x01, symbol Switch:SW_DIP_x01
- removed U10: TPS61240, symbol Power_Management:TPS61240
- removed U11: LTC4054, symbol Power_Management:LTC4054
- removed U12, U13: FP6134-33S5, symbol Power_Management:FP6134-33S5
- removed U4: 74HC4066N, DIP254P762X420-14, symbol 74HC4066N:74HC4066N
- removed U5: MP20046, symbol MP:MP20046
- removed U6: BQ25895RTW, Package_DFN_QFN:Texas_S-PWQFN-N24_EP2.7x2.7mm_ThermalVias, symbol Battery_Management:BQ25895RTW
- removed U7: TPS61088RHLR, IC_TPS61088RHLR, symbol TPS61088RHLR:TPS61088RHLR
- removed U8: PW5300, symbol Power_Management:PW5300
- removed U9: PW2053, symbol Power_Management:PW2053
- added C10, C13, C9: 47U, symbol Device:C
- added C24: 1N, symbol Device:C
- added D1: SS34, Diode_SMD:D_1210_3225Metric, symbol Diode:1N914
- added D3, D4: LED, symbol Device:LED
- added D6: SS34, Diode_THT:D_DO-35_SOD27_P7.62mm_Horizontal, symbol Diode:1N914
- added R1: PROG, Resistor_SMD:R_0603_1608Metric, symbol Device:R
- added R3, R4: 1K, Resistor_SMD:R_0603_1608Metric, symbol Device:R
- added RV1: 10K, symbol Device:R_Potentiometer
- added SW1: SW_MEC_5G, symbol Switch:SW_MEC_5G
- added SW2: SW_DIP_x01, symbol Switch:SW_DIP_x01
- added U1: TC4056A, TC4056A:SOP-8_L4.9-W3.9-P1.27-LS6.0-BL-EP, symbol kicad_lceda:TC4056A
- added U3: MT3608, Package_TO_SOT_SMD:SOT-23-6, symbol Regulator_Switching:MT3608
- added U9: SL2.1S, SL2.1:SSOP-16_L4.6-W2.6-P0.53-LS4.0-BL, symbol SL2.1S:SL2.1S
- added Y3: 12M, symbol Device:Crystal_Small
- C1: renamed from C3; value 10U -> 100n
- C15: renamed from C17; value 1u -> 47U
- C18: renamed from C10; value 100p -> 47p
- C20: renamed from C12; value 5n6 -> 2.2n
- C21: renamed from C13; value 5n6 -> 1n
- C22: renamed from C14; value 180p -> NC
- C23: value 1u -> 100N
- C25: value 0.1u -> 22p
- C26: value 1u -> 22p
- C28: renamed from C19; value 22n -> 6.8n
- C30: value 22U -> 100n
- C4, C5: value 0.1U -> 100n
- C6: renamed from C9; value 0.1U -> 100n
- L1: value 120uH -> 22U
- R10: renamed from R?; value 5.1k -> 12k; footprint (none) -> Resistor_SMD:R_0603_1608Metric
- R11, R12, R13, R8, R9: renamed from R?; footprint (none) -> Resistor_SMD:R_0603_1608Metric
- R14: renamed from R9; value 10 -> 100; footprint (none) -> Resistor_SMD:R_0603_1608Metric
- R15: value 100k -> 22; footprint (none) -> Resistor_SMD:R_0603_1608Metric
- R16: value 1k -> 22; footprint (none) -> Resistor_SMD:R_0603_1608Metric
- R17: value 88K -> 4.7k; footprint (none) -> Resistor_SMD:R_0603_1608Metric
- R2: renamed from R1; footprint (none) -> Resistor_SMD:R_0603_1608Metric
- R5: renamed from R3; footprint (none) -> Resistor_SMD:R_0603_1608Metric
- R6: renamed from R4; footprint (none) -> Resistor_SMD:R_0603_1608Metric
- R7: value 47k -> 2.2k; footprint (none) -> Resistor_SMD:R_0603_1608Metric
- U4: renamed from U?; footprint kicad_lceda:WIRELM-SMD_E01-ML01S -> e01:WIRELM-SMD_E01-ML01S
- U7: renamed from U?; footprint kicad_lceda:WIFIM-SMD_ESP-12F-ESP8266MOD -> esp8266:WIFIM-SMD_ESP-12F-ESP8266MOD
- U8: renamed from U?; footprint kicad_lceda:WIRELM-SMD_E07-M1101S -> e07:WIRELM-SMD_E07-M1101S
- Y2: renamed from Y?; value Crystal_Small -> 12M
- gave numbers to parts that had none: 7
- renumbered C33 to C17, C11 to C19, C20 to C27, C21 to C29, C1 to C3, C6 to C7, C7 to C8, D4 to D5, D3 to D7, D2 to D8, U3 to U10, U1 to U2, U14 to U5, U2 to U6
Connections:
- net A0_GDO0_1 is gone; now on net A0_NRF_CS: U2.36 (PF7)
- net A1_RE_CS_1 is gone; now on net A1_NRF_CE: U2.37 (PF6)
- net A2_GDO0_2 is gone; now on net A2_RF_GDO0: U2.38 (PF5)
- net A3_RE_CS_2 is gone; now on net A3_RF_CS: U2.39 (PF4)
- net AGND is gone; now on an unnamed net: U10.11 (AGND)
- net BMISO is gone; now on net MISO: U7.18 (MISO)
- net BMOSI is gone; now on net MOSI: U7.21 (MOSI)
- net D6 is gone; now on net MOD: U2.27 (PD7)
- net D7 is gone; now on net D7_IRQ: U2.1 (PE6)
- net DEMOD_OUT is gone; now on net ID_OUT: U10.13 (DEMOD_OUT)
- net IO13 is gone; now on net PB7: U2.32 (PC7)
- net ISP_RST is gone; now on net ARST: R2.1, U2.13 (~{RESET})
- net RF_GDO2_2 is gone; now on net D2_RF_GDO2: U2.19 (PD1)
- net RXD is gone; now on net ATX: U2.21 (PD3)
- net TXD is gone; now on net ARX: U2.20 (PD2)
- net VBUS_5V_IN is gone; now on net GND: C25.1, C26.1
- net +3V3: no longer C23.1, R15.2, R7.1
- net +5V: now also C23.1, R7.1, C10.1, C13.1, C24.1, D1.1 (K), D6.1 (K); no longer C17.1, F1.1, R17.1, U2.7 (VBUS)
- net ARST: now also SW1.1 (A), SW1.2 (A)
- net BAT: now also L1.1, C9.2, SW2.1, U1.5 (BAT), U3.5 (IN)
- net CHUD+: now also U9.2 (DP2)
- net CHUD-: now also U9.1 (DM2)
- net LB1: no longer L1.1
- net LB2: no longer L1.2
- net RD_N: now also R16.2; no longer D8.2 (A2)
- net RD_P: now also R15.1; no longer D7.2 (A2)
- net at R7.2: now also RV1.1, U3.3 (FB)
- net GND: now reaches R17.2
- net GND: now also C1.2, C11.1, C12.1, C14.1, C15.2, C16.2, C17.2, C19.2, C2.1, C23.2, C28.1, C29.2, C3.2, C30.2, C4.2, C5.2, C6.2, C7.1, C8.1, D2.6 (VSS), D5.1 (K), D7.1 (A1), D8.1 (A1), J1.5 (GND), R6.2, U10.1 (VSS), U10.5 (DVSS), U2.15 (GND), U2.23 (GND), U2.35 (GND), U2.43 (GND), U2.45 (GND), U2.5 (UGND), U4.8 (GND), U5.1 (GND), U6.1 (GND), U7.9 (GND), U8.8 (GND), Y1.2, Y1.4, C10.2, C13.2, C24.2, C9.1, R1.1, RV1.2, RV1.3, SW1.3 (B), SW1.4 (B), U1.1 (TEMP), U1.3 (GND), U1.9 (EP), U3.2 (GND), U9.8 (VSS)
- net at R16.1: now also U9.4 (DP1)
- net GPIO9: now reaches U7.19 (GPIO9)
- net GPIO10: now reaches U7.20 (GPIO10)
- net UDP: now reaches J1.3 (D+)
- net UDP: now also D7.2 (A2), U9.6 (UDP)
- net UDM: now reaches J1.2 (D-)
- net UDM: now also D8.2 (A2), U9.5 (UDM)
- net PB0: now reaches U2.8 (PB0)
- net 3V~24V: no longer names the net of C30.1
- net A4 renamed PF1
- net A5 renamed PF0
- net ANT1: no longer names the net of R14.2, U10.3 (ANT1)
- net ANT2: no longer names the net of C20.1, C21.2, C22.2, U10.6 (ANT2)
- net BCS renamed CS0
- net BSCK renamed SCLK
- net CDEC_IN: no longer names the net of C27.1, U10.10 (CDEC_IN)
- net CDEC_OUT: no longer names the net of C27.2, U10.9 (CDEC_OUT)
- net D4 renamed PD4
- net D5 renamed ID_OUT
- net DC2: no longer names the net of U10.16 (DC2)
- net DC2: now also C28.2; no longer C28.1
- net DEMOD_IN: no longer names the net of C18.2, C19.1, U10.8 (DEMOD_IN)
- removed net Earth: C1.2, C11.1, C12.1, C14.1, C15.2, C16.2, C17.2, C19.2, C2.1, C23.2, C25.2, C26.2, C28.2, C29.2, C3.2, C30.2, C4.2, C5.2, C6.2, C7.1, C8.1, D2.6 (VSS), D5.1 (K), D7.1 (A1), D8.1 (A1), J1.5 (GND), R16.2, R6.2, U10.1 (VSS), U10.14 (SHD), U10.5 (DVSS), U2.15 (GND), U2.23 (GND), U2.35 (GND), U2.43 (GND), U2.45 (GND), U2.5 (UGND), U4.8 (GND), U5.1 (GND), U6.1 (GND), U7.9 (GND), U8.8 (GND), Y1.2, Y1.4
- net FCAP: no longer names the net of C29.1, U10.15 (FCAP)
- net IICSCL renamed GPIO4
- net IICSDA renamed GPIO5
- net IO10 renamed PB6
- net IO11 renamed PB7
- net IO12 renamed PD6
- net IO8 renamed OPEN_CC1101
- net IO9 renamed SHD
- net SHD: now also R17.1, U10.14 (SHD)
- net ISP_MISO renamed AMOSI
- net ISP_MOSI renamed AMISO
- net ISP_SCK renamed ASCK
- net RF_GDO2_1 renamed PD0
- new net: R15.2, U9.3 (DM1)
- new net: R3.1, U1.7 (CHRG)
- new net: D3.1 (K), R3.2
- new net: R1.2, U1.2 (PROG)
- new net: R4.1, U1.6 (STDBY)
- new net: C25.2, U9.12 (XIN), Y3.1
- new net: C26.2, U9.11 (XOUT), Y3.2
- new net: D4.1 (K), R4.2
- new net: SW2.2, U3.4 (EN)
- new net: D6.2 (A), L1.2, U3.1 (SW)
- new net DM3-: U9.15 (DM3)
- new net DM4-: U9.13 (DM4)
- new net DP3+: U9.16 (DP3)
- new net DP4+: U9.14 (DP4)
- new net SL_1.8V: U9.10 (VDD18)
- new net SL_3.3V: U9.9 (VDD33)
- new net VBUS: C17.1, D1.2 (A), D3.2 (A), D4.2 (A), F1.1, U1.4 (VCC), U1.8 (CE), U2.7 (VBUS), U9.7 (VDD5)
- no-connect marks 14 -> 10
Other:
- note added: "4.2V-5V"
- note added: "5V-3.3V"
- note added: "ATmega32U4RC-M"
- note added: "CC1101"
- note added: "CH340G_ESP8266"
- note added: "EM4095"
- note added: "ESP8266"
- note added: "POWER_LI_LON"
- note added: "USB"
- note added: "USB_HUP"
- note added: "WS2812_LED"
- note added: "nRF2.4G"
- note removed: "POWER"
- note removed: "RF_POWER_SWITCH"
- note removed: "SPI_SEL"
- moved on the sheet: C1, C11, C12, C14, C15, C16, C17, C18, C19, C2, C20, C21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
